File: schinkli_brain.kicad_pcb (KiCad board)
At the start: 2 copper layers, 40 x 30 mm, 9 parts, among them J1 BridgeHeader, J3_1 VMOT, Q2 WE-FDSM3.3, U1 ESP-12E

Commit message: add 3d image and update readme
Parts:
- J1: footprint Connector_PinHeader_2.54mm:PinHeader_1x06_P2.54mm_Vertical -> Connector_PinSocket_2.54mm:PinSocket_1x06_P2.54mm_Vertical; moved to B.Cu
- turned J1 to 180 degrees
Changed lines of the file:
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@@
     (add_net VCC)
+  )
+  (module Connector_PinSocket_2.54mm:PinSocket_1x06_P2.54mm_Vertical (layer B.Cu)
+    (at 53.5 108.5 180)
+    (descr "Through hole straight socket strip, 1x06, 2.54mm pitch, single row (from Kicad 4.0.7), script generated")
+    (tags "Through hole socket strip THT 1x06 2.54mm single row")
+    (fp_text reference J1 (at -2.484 1.388) (layer B.SilkS)
+      (effects (font (size 1 1) (thickness 0.15)) (justify mirror))
+    )
+    (fp_text value BridgeHeader (at 0 -15.03) (layer B.Fab)
+      (effects (font (size 1 1) (thickness 0.15)) (justify mirror))
+    )
+    (fp_text user %R (at 0 -6.35 270) (layer B.Fab)
+      (effects (font (size 1 1) (thickness 0.15)) (justify mirror))
+    )
+    (fp_line (start -1.8 -14.45) (end -1.8 1.8) (layer B.CrtYd) (width 0.05))
+    (fp_line (start 1.75 -14.45) (end -1.8 -14.45) (layer B.CrtYd) (width 0.05))
+    (fp_line (start 1.75 1.8) (end 1.75 -14.45) (layer B.CrtYd) (width 0.05))
+    (fp_line (start -1.8 1.8) (end 1.75 1.8) (layer B.CrtYd) (width 0.05))
+    (fp_line (start 0 1.33) (end 1.33 1.33) (layer B.SilkS) (width 0.12))
+    (fp_line (start 1.33 1.33) (end 1.33 0) (layer B.SilkS) (width 0.12))
+    (fp_line (start 1.33 -1.27) (end 1.33 -14.03) (layer B.SilkS) (width 0.12))
+    (fp_line (start -1.33 -14.03) (end 1.33 -14.03) (layer B.SilkS) (width 0.12))
+    (fp_line (start -1.33 -1.27) (end -1.33 -14.03) (layer B.SilkS) (width 0.12))
+    (fp_line (start -1.33 -1.27) (end 1.33 -1.27) (layer B.SilkS) (width 0.12))
+    (fp_line (start -1.27 -13.97) (end -1.27 1.27) (layer B.Fab) (width 0.1))
+    (fp_line (start 1.27 -13.97) (end -1.27 -13.97) (layer B.Fab) (width 0.1))
+    (fp_line (start 1.27 0.635) (end 1.27 -13.97) (layer B.Fab) (width 0.1))
+    (fp_line (start 0.635 1.27) (end 1.27 0.635) (layer B.Fab) (width 0.1))
+    (fp_line (start -1.27 1.27) (end 0.635 1.27) (layer B.Fab) (width 0.1))
+    (pad 6 thru_hole oval (at 0 -12.7 180) (size 1.7 1.7) (drill 1) (layers *.Cu *.Mask)
+      (net 2 DP4))
+    (pad 5 thru_hole oval (at 0 -10.16 180) (size 1.7 1.7) (drill 1) (layers *.Cu *.Mask)
+      (net 3 DP3))
+    (pad 4 thru_hole oval (at 0 -7.62 180) (size 1.7 1.7) (drill 1) (layers *.Cu *.Mask)
+      (net 4 DP2))
+    (pad 3 thru_hole oval (at 0 -5.08 180) (size 1.7 1.7) (drill 1) (layers *.Cu *.Mask)
+      (net 5 DP1))
+    (pad 2 thru_hole oval (at 0 -2.54 180) (size 1.7 1.7) (drill 1) (layers *.Cu *.Mask)
+      (net 1 GND))
+    (pad 1 thru_hole rect (at 0 0 180) (size 1.7 1.7) (drill 1) (layers *.Cu *.Mask)
+      (net 6 VCC))
+    (model ${KISYS3DMOD}/Connector_PinSocket_2.54mm.3dshapes/PinSocket_1x06_P2.54mm_Vertical.wrl
+      (at (xyz 0 0 0))
+      (scale (xyz 1 1 1))
+      (rotate (xyz 0 0 0))
+    )
   )
   (module MountingHole:MountingHole_3.2mm_M3 (layer F.Cu)
@@
     (pad 1 np_thru_hole circle (at 0 0) (size 3.2 3.2) (drill 3.2) (layers *.Cu *.Mask))
   )
-  (module Connector_PinHeader_2.54mm:PinHeader_1x06_P2.54mm_Vertical (layer F.Cu)
-    (at 53.5 108.5)
-    (descr "Through hole straight pin header, 1x06, 2.54mm pitch, single row")
-    (tags "Through hole pin header THT 1x06 2.54mm single row")
-    (fp_text reference J1 (at -2.484 -1.388) (layer F.SilkS)
-      (effects (font (size 1 1) (thickness 0.15)))
-    )
-    (fp_text value BridgeHeader (at 0 15.03) (layer F.Fab)
-      (effects (font (size 1 1) (thickness 0.15)))
-    )
-    (fp_text user %R (at 0 6.35 90) (layer F.Fab)
-      (effects (font (size 1 1) (thickness 0.15)))
-    )
-    (fp_line (start 1.8 -1.524) (end -1.8 -1.524) (layer F.CrtYd) (width 0.05))
-    (fp_line (start 1.8 14.5) (end 1.8 -1.524) (layer F.CrtYd) (width 0.05))
-    (fp_line (start -1.8 14.5) (end 1.8 14.5) (layer F.CrtYd) (width 0.05))
-    (fp_line (start -1.8 -1.524) (end -1.8 14.5) (layer F.CrtYd) (width 0.05))
-    (fp_line (start -1.33 -1.33) (end 0 -1.33) (layer F.SilkS) (width 0.12))
-    (fp_line (start -1.33 0) (end -1.33 -1.33) (layer F.SilkS) (width 0.12))
-    (fp_line (start -1.33 1.27) (end 1.33 1.27) (layer F.SilkS) (width 0.12))
-    (fp_line (start 1.33 1.27) (end 1.33 14.03) (layer F.SilkS) (width 0.12))
-    (fp_line (start -1.33 1.27) (end -1.33 14.03) (layer F.SilkS) (width 0.12))
-    (fp_line (start -1.33 14.03) (end 1.33 14.03) (layer F.SilkS) (width 0.12))
-    (fp_line (start -1.27 -0.635) (end -0.635 -1.27) (layer F.Fab) (width 0.1))
-    (fp_line (start -1.27 13.97) (end -1.27 -0.635) (layer F.Fab) (width 0.1))
-    (fp_line (start 1.27 13.97) (end -1.27 13.97) (layer F.Fab) (width 0.1))
-    (fp_line (start 1.27 -1.27) (end 1.27 13.97) (layer F.Fab) (width 0.1))
-    (fp_line (start -0.635 -1.27) (end 1.27 -1.27) (layer F.Fab) (width 0.1))
-    (pad 6 thru_hole oval (at 0 12.7) (size 1.7 1.7) (drill 1) (layers *.Cu *.Mask)
-      (net 2 DP4))
-    (pad 5 thru_hole oval (at 0 10.16) (size 1.7 1.7) (drill 1) (layers *.Cu *.Mask)
-      (net 3 DP3))
-    (pad 4 thru_hole oval (at 0 7.62) (size 1.7 1.7) (drill 1) (layers *.Cu *.Mask)
-      (net 4 DP2))
-    (pad 3 thru_hole oval (at 0 5.08) (size 1.7 1.7) (drill 1) (layers *.Cu *.Mask)
-      (net 5 DP1))
-    (pad 2 thru_hole oval (at 0 2.54) (size 1.7 1.7) (drill 1) (layers *.Cu *.Mask)
-      (net 1 GND))
-    (pad 1 thru_hole rect (at 0 0) (size 1.7 1.7) (drill 1) (layers *.Cu *.Mask)
-      (net 6 VCC))
-    (model ${KISYS3DMOD}/Connector_PinHeader_2.54mm.3dshapes/PinHeader_1x06_P2.54mm_Vertical.wrl
-      (at (xyz 0 0 0))
-      (scale (xyz 1 1 1))
-      (rotate (xyz 0 0 0))
-    )
-  )
   (module Symbol:wilmas_playground_8mm (layer F.Cu)
